Commit message: Update arduinobot.urdf.xacro

File: Section4_Digital_Twin/arduinobot_ws/src/arduinobot_description/urdf/arduinobot.urdf.xacro (robot description, xacro)
@@ -130,5 +130,4 @@
         </collision>
     </link>
-    <link name="tool_link"></link>
     <!-- Joints -->
     <joint name="virtual_joint" type="fixed">
@@ -183,8 +182,3 @@
         <mimic joint="joint_4" multiplier="-1"/>
     </joint>
-    <joint name ="gripper_right_to_tool" type="fixed">
-        <parent link="gripper_right"/>
-        <child link = "tool_link"/>
-        <origin xyz="0 0 0"/>
-    </joint>
 </robot>

Commit message: removed useless variables

File: Section4_Digital_Twin/arduinobot_ws/src/arduinobot_description/urdf/arduinobot.urdf.xacro (robot description, xacro)
@@ -1,16 +1,8 @@
 <?xml version="1.0"?>
 <robot xmlns:xacro="http://www.ros.org/wiki/xacro" name="arduinobot">
-    <!-- Load Simulated or Real Hardware Interfaces -->
-    <xacro:arg name="is_sim" default="true"/>
     <!-- Useful XACRO Variables (Properties) -->
     <xacro:property name="PI" value="3.14159265359" />
     <xacro:property name="effort" value="30.0" />
     <xacro:property name="velocity" value="10.0" />
-    <xacro:property name="joint_arm_lower_limit" value="-${PI / 2}" />
-    <xacro:property name="joint_arm_upper_limit" value="${PI / 2}" />
-    <xacro:property name="joint_finger_right_lower_limit" value="-${PI / 2}" />
-    <xacro:property name="joint_finger_right_upper_limit" value="0.0" />
-    <xacro:property name="joint_finger_left_lower_limit" value="0.0" />
-    <xacro:property name="joint_finger_left_upper_limit" value="${PI / 2}" />
     <!-- Useful Macros -->
     <xacro:macro name="default_inertial" params="mass">
@@ -141,5 +133,5 @@
         <origin xyz="0 0 0.307"/>
         <axis xyz="0 0 1"/>
-        <limit lower="${joint_arm_lower_limit}" upper="${joint_arm_upper_limit}"
+        <limit lower="-${PI / 2}" upper="${PI / 2}"
                effort="${effort}" velocity="${velocity}"/>
     </joint>
@@ -149,5 +141,5 @@
         <origin xyz="-0.02 0 0.35"/>
         <axis xyz="1 0 0"/>
-        <limit lower="${joint_arm_lower_limit}" upper="${joint_arm_upper_limit}"
+        <limit lower="-${PI / 2}" upper="${PI / 2}"
                 effort="${effort}" velocity="${velocity}"/>
     </joint>
@@ -157,5 +149,5 @@
         <origin xyz="0 0 0.8"/>
         <axis xyz="1 0 0"/>
-        <limit lower="${joint_arm_lower_limit}" upper="${joint_arm_upper_limit}"
+        <limit lower="-${PI / 2}" upper="${PI / 2}"
                effort="${effort}" velocity="${velocity}"/>
     </joint>
@@ -170,5 +162,5 @@
         <origin xyz="-0.04 0.13 -0.1"/>
         <axis xyz="0 0 1"/>
-        <limit lower="${joint_finger_right_lower_limit}" upper="${joint_finger_right_upper_limit}"
+        <limit lower="-${PI / 2}" upper="0.0"
                effort="${effort}" velocity="${velocity}"/>
     </joint>
@@ -178,5 +170,5 @@
         <origin xyz="-0.22 0.13 -0.1"/>
         <axis xyz="0 0 1"/>
-        <limit lower="${joint_finger_left_lower_limit}" upper="${joint_finger_left_upper_limit}"
+        <limit lower="0.0" upper="${PI / 2}"
                effort="${effort}" velocity="${velocity}"/>
         <mimic joint="joint_4" multiplier="-1"/>

File: Section5_Control/arduinobot_ws/src/arduinobot_description/urdf/arduinobot.urdf.xacro (robot description, xacro)
@@ -1,10 +1,12 @@
 <?xml version="1.0"?>
 <robot xmlns:xacro="http://www.ros.org/wiki/xacro" name="arduinobot">
-    <!-- Include XACRO Variables -->
-    <xacro:include filename="$(find arduinobot_description)/urdf/arduinobot_variables.xacro" />
     <!-- Include Gazebo Parameters -->
     <xacro:include filename="$(find arduinobot_description)/urdf/arduinobot_gazebo.xacro" />
     <!-- Include ros2_control Plugins -->
     <xacro:include filename="$(find arduinobot_description)/urdf/arduinobot_ros2_control.xacro" />
+    <!-- Useful XACRO Variables (Properties) -->
+    <xacro:property name="PI" value="3.14159265359" />
+    <xacro:property name="effort" value="30.0" />
+    <xacro:property name="velocity" value="10.0" />
     <!-- Useful Macros -->
     <xacro:macro name="default_inertial" params="mass">
@@ -133,5 +135,4 @@
         </collision>
     </link>
-    <link name="tool_link"></link>
     <!-- Joints -->
     <joint name="virtual_joint" type="fixed">
@@ -145,5 +146,5 @@
         <origin xyz="0 0 0.307"/>
         <axis xyz="0 0 1"/>
-        <limit lower="${joint_arm_lower_limit}" upper="${joint_arm_upper_limit}"
+        <limit lower="-${PI / 2}" upper="${PI / 2}"
                effort="${effort}" velocity="${velocity}"/>
     </joint>
@@ -153,5 +154,5 @@
         <origin xyz="-0.02 0 0.35"/>
         <axis xyz="1 0 0"/>
-        <limit lower="${joint_arm_lower_limit}" upper="${joint_arm_upper_limit}"
+        <limit lower="-${PI / 2}" upper="${PI / 2}"
                 effort="${effort}" velocity="${velocity}"/>
     </joint>
@@ -161,5 +162,5 @@
         <origin xyz="0 0 0.8"/>
         <axis xyz="1 0 0"/>
-        <limit lower="${joint_arm_lower_limit}" upper="${joint_arm_upper_limit}"
+        <limit lower="-${PI / 2}" upper="${PI / 2}"
                effort="${effort}" velocity="${velocity}"/>
     </joint>
@@ -174,5 +175,5 @@
         <origin xyz="-0.04 0.13 -0.1"/>
         <axis xyz="0 0 1"/>
-        <limit lower="${joint_finger_right_lower_limit}" upper="${joint_finger_right_upper_limit}"
+        <limit lower="-${PI / 2}" upper="0.0"
                effort="${effort}" velocity="${velocity}"/>
     </joint>
@@ -182,12 +183,7 @@
         <origin xyz="-0.22 0.13 -0.1"/>
         <axis xyz="0 0 1"/>
-        <limit lower="${joint_finger_left_lower_limit}" upper="${joint_finger_left_upper_limit}"
+        <limit lower="0.0" upper="${PI / 2}"
                effort="${effort}" velocity="${velocity}"/>
         <mimic joint="joint_4" multiplier="-1"/>
-    </joint>
-    <joint name ="gripper_right_to_tool" type="fixed">
-        <parent link="gripper_right"/>
-        <child link = "tool_link"/>
-        <origin xyz="0 0 0"/>
     </joint>
     <!-- Transmissions-->

File: Section5_Control/arduinobot_ws/src/arduinobot_description/urdf/arduinobot_ros2_control.xacro (robot description, xacro)
@@ -1,7 +1,6 @@
 <?xml version="1.0"?>
 <robot xmlns:xacro="http://www.ros.org/wiki/xacro" name="arduinobot">
-    <!-- Include XACRO Variables -->
-    <xacro:include filename="$(find arduinobot_description)/urdf/arduinobot_variables.xacro" />
     <ros2_control name="RobotSystem" type="system">
+        <xacro:property name="PI" value="3.14159265359" />
         <!-- ros2_control Gazebo -->
         <hardware>
@@ -10,6 +9,6 @@
         <joint name="joint_1">
             <command_interface name="position">
-            <param name="min">${joint_arm_lower_limit}</param>
-            <param name="max">${joint_arm_upper_limit}</param>
+            <param name="min">-${PI / 2}</param>
+            <param name="max">${PI / 2}</param>
             </command_interface>
             <state_interface name="position"/>
@@ -17,6 +16,6 @@
         <joint name="joint_2">
             <command_interface name="position">
-            <param name="min">${joint_arm_lower_limit}</param>
-            <param name="max">${joint_arm_upper_limit}</param>
+            <param name="min">-${PI / 2}</param>
+            <param name="max">${PI / 2}</param>
             </command_interface>
             <state_interface name="position"/>
@@ -24,6 +23,6 @@
         <joint name="joint_3">
             <command_interface name="position">
-            <param name="min">${joint_arm_lower_limit}</param>
-            <param name="max">${joint_arm_upper_limit}</param>
+            <param name="min">-${PI / 2}</param>
+            <param name="max">${PI / 2}</param>
             </command_interface>
             <state_interface name="position"/>
@@ -31,6 +30,6 @@
         <joint name="joint_4">
             <command_interface name="position">
-            <param name="min">${joint_finger_right_lower_limit}</param>
-            <param name="max">${joint_finger_right_upper_limit}</param>
+            <param name="min">-${PI / 2}</param>
+            <param name="max">0.0</param>
             </command_interface>
             <state_interface name="position"/>
@@ -40,6 +39,6 @@
             <param name="multiplier">-1</param>
             <command_interface name="position">
-            <param name="min">${joint_finger_left_lower_limit}</param>
-            <param name="max">${joint_finger_left_upper_limit}</param>
+            <param name="min">0.0</param>
+            <param name="max">${PI / 2}</param>
             </command_interface>
         </joint>
